Commit message: Support side-mounted arm configuration

File: src/fr3_real_bringup/urdf/robot.urdf.xacro (robot description, xacro)
@@ -16,4 +16,7 @@
   <xacro:property name="b" value="${cfg['base']}"/>
   <xacro:property name="g" value="${cfg['tool']}"/>
+  <xacro:property name="base_parent" value="${'table' if b.get('mounting', 'tabletop') == 'tabletop' else 'world'}"/>
+  <xacro:property name="base_z" value="${t['height'] if b.get('mounting', 'tabletop') == 'tabletop' else b['z']}"/>
+  <xacro:property name="base_rpy" value="${[0, 0, b['yaw']] if b.get('mounting', 'tabletop') == 'tabletop' else [b['roll'], b['pitch'], b['yaw']]}"/>
   <xacro:property name="gripper_closed_position" value="$(arg gripper_closed_position)"/>
   <xacro:include filename="$(arg arm_file)"/>
@@ -47,6 +50,6 @@
   </joint>
   <joint name="table_to_base" type="fixed">
-    <parent link="table"/><child link="base_link"/>
-    <origin xyz="${b['x']} ${b['y']} ${t['height']}" rpy="0 0 ${b['yaw']}"/>
+    <parent link="${base_parent}"/><child link="base_link"/>
+    <origin xyz="${b['x']} ${b['y']} ${base_z}" rpy="${' '.join(map(str,base_rpy))}"/>
   </joint>
   <link name="tool0"/>
